File: hardware/next-micro.kicad_pcb (KiCad board)
At the start: 2 copper layers, 17.8 x 33 mm, 26 parts, among them J1 USB_C_Receptacle_USB2.0, J2 Conn_01x13, J3 Conn_01x05, J4 Conn_01x13, SW1 RESET, U1 ATmega32U4-M, U2 RT9013-33GB, Y1 8MHz

Commit message: Add PCBA files and move files
Parts:
- J1: footprint rp-micro:USB Type-C Mid-Mount Receptacle 16P -> next_micro:USB Type-C Mid-Mount Receptacle 16P
