File: hardware/next-micro.kicad_sch (KiCad schematic)
At the start: 25 parts, among them J1 USB_C_Receptacle_USB2.0, J2 Conn_01x13, J3 Conn_01x05, J4 Conn_01x13, SW1 RESET, U1 ATmega32U4-M, U2 RT9013-33GB, Y1 8MHz

Commit message: Add PCBA files and move files
Parts:
- J1: footprint rp-micro:USB Type-C Mid-Mount Receptacle 16P -> next_micro:USB Type-C Mid-Mount Receptacle 16P
- JP1: Note (none) -> LDO Bypass
Other:
- title: (none) -> Next Micro
- moved on the sheet: C1, C2, C3, C4, C5, C6, C7, C8, C9, D1, F1, J1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

Commit message: Replace D1 footprint to hand soldering version
Parts:
- D1: footprint Diode_SMD:D_SOD-323 -> Diode_SMD:D_SOD-323_HandSoldering
Changed lines of the file:
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@@
     (property "Reference" "D1" (id 0) (at 218.7575 43.18 0))
     (property "Value" "B5817" (id 1) (at 218.7575 45.72 0))
-    (property "Footprint" "Diode_SMD:D_SOD-323" (id 2) (at 218.44 45.085 0)
+    (property "Footprint" "Diode_SMD:D_SOD-323_HandSoldering" (id 2) (at 218.44 45.085 0)
       (effects (font (size 1.27 1.27)) hide)
     )
@@
     (in_bom no) (on_board yes)
     (property "Reference" "JP1" (id 0) (at 242.57 26.67 0))
-    (property "Value" "SolderJumper_2_Open" (id 1) (at 242.57 29.21 0))
+    (property "Value" "SolderJumper_2_Open" (id 1) (at 242.57 26.67 0)
+      (effects (font (size 1.27 1.27)) hide)
+    )
     (property "Footprint" "Jumper:SolderJumper-2_P1.3mm_Open_TrianglePad1.0x1.5mm" (id 2) (at 242.57 33.02 0)
       (effects (font (size 1.27 1.27)) hide)
@@
       (effects (font (size 1.27 1.27)) hide)
     )
-    (property "Note" "LDO Bypass" (id 4) (at 242.57 35.56 0))
+    (property "Note" "LDO Bypass" (id 4) (at 242.57 29.21 0))
     (pin "1")
     (pin "2")
@@
     )
     (path "/1169cf00-fc1c-4b97-a593-f21f2b3caa7b"
-      (reference "D1") (unit 1) (value "B5817") (footprint "Diode_SMD:D_SOD-323")
+      (reference "D1") (unit 1) (value "B5817") (footprint "Diode_SMD:D_SOD-323_HandSoldering")
     )
     (path "/c4f10a29-86cd-410e-967a-7c8a03890ef2"
